Commit message: centralize load_robot func

File: examples/ur10/data/robot.urdf (robot description, URDF)
Before this commit: robot ur10e, 29 links, 28 joints
Links:
- link ur10e_d435_mount_link: geometry collision mesh filename=package://agimus-demos/meshes/ur10e_d435_mount.stl; visual mesh filename=package://agimus-demos/meshes/ur10e_d435_mount.stl
- link ur10e_tool_link: geometry collision cylinder length=0.25 radius=0.0015; collision mesh filename=package://agimus-demos/meshes/ur10e_tip.stl
